Commit message: For real this time

File: robots/g1_description/g1_23dof.urdf (robot description, URDF)
Before this commit: robot g1_23dof, 32 links, 31 joints
Links:
- removed link d435_link
- removed link mid360_link
Joints:
- removed joint d435_joint
- removed joint mid360_joint

File: robots/g1_description/g1_29dof.urdf (robot description, URDF)
Before this commit: robot g1_29dof, 39 links, 38 joints
Links:
- removed link d435_link
- removed link mid360_link
- added link world
- link head_link: geometry collision mesh filename=package://g1_description/meshes/head_link.STL; visual mesh filename=package://g1_description/meshes/head_link.STL
- link left_ankle_pitch_link: geometry collision mesh filename=package://g1_description/meshes/left_ankle_pitch_link.STL; visual mesh filename=package://g1_description/meshes/left_ankle_pitch_link.STL
- link left_ankle_roll_link: geometry collision sphere radius=0.005; collision sphere radius=0.005
- link left_elbow_link: geometry collision mesh filename=package://g1_description/meshes/left_elbow_link.STL; visual mesh filename=package://g1_description/meshes/left_elbow_link.STL
- link left_hip_pitch_link: geometry collision mesh filename=package://g1_description/meshes/left_hip_pitch_link.STL; visual mesh filename=package://g1_description/meshes/left_hip_pitch_link.STL
- link left_hip_roll_link: geometry collision mesh filename=package://g1_description/meshes/left_hip_roll_link.STL; visual mesh filename=package://g1_description/meshes/left_hip_roll_link.STL
- link left_hip_yaw_link: geometry collision mesh filename=package://g1_description/meshes/left_hip_yaw_link.STL; visual mesh filename=package://g1_description/meshes/left_hip_yaw_link.STL
- link left_knee_link: geometry collision mesh filename=package://g1_description/meshes/left_knee_link.STL; visual mesh filename=package://g1_description/meshes/left_knee_link.STL
- link left_rubber_hand: geometry visual mesh filename=package://g1_description/meshes/left_rubber_hand.STL
- link left_shoulder_pitch_link: geometry collision cylinder length=0.05 radius=0.03; visual mesh filename=package://g1_description/meshes/left_shoulder_pitch_link.STL
- link left_shoulder_roll_link: geometry collision cylinder length=0.03 radius=0.03; visual mesh filename=package://g1_description/meshes/left_shoulder_roll_link.STL
- link left_shoulder_yaw_link: geometry collision mesh filename=package://g1_description/meshes/left_shoulder_yaw_link.STL; visual mesh filename=package://g1_description/meshes/left_shoulder_yaw_link.STL
- link left_wrist_pitch_link: geometry collision mesh filename=package://g1_description/meshes/left_wrist_pitch_link.STL; visual mesh filename=package://g1_description/meshes/left_wrist_pitch_link.STL
- link left_wrist_roll_link: geometry collision mesh filename=package://g1_description/meshes/left_wrist_roll_link.STL; visual mesh filename=package://g1_description/meshes/left_wrist_roll_link.STL
- link left_wrist_yaw_link: geometry collision mesh filename=package://g1_description/meshes/left_wrist_yaw_link.STL; visual mesh filename=package://g1_description/meshes/left_wrist_yaw_link.STL
- link logo_link: geometry collision mesh filename=package://g1_description/meshes/logo_link.STL; visual mesh filename=package://g1_description/meshes/logo_link.STL
- link pelvis: geometry visual mesh filename=package://g1_description/meshes/pelvis.STL
- link pelvis_contour_link: geometry collision mesh filename=package://g1_description/meshes/pelvis_contour_link.STL; visual mesh filename=package://g1_description/meshes/pelvis_contour_link.STL
- link right_ankle_pitch_link: geometry collision mesh filename=package://g1_description/meshes/right_ankle_pitch_link.STL; visual mesh filename=package://g1_description/meshes/right_ankle_pitch_link.STL
- link right_ankle_roll_link: geometry collision sphere radius=0.005; collision sphere radius=0.005
- link right_elbow_link: geometry collision mesh filename=package://g1_description/meshes/right_elbow_link.STL; visual mesh filename=package://g1_description/meshes/right_elbow_link.STL
- link right_hip_pitch_link: geometry collision mesh filename=package://g1_description/meshes/right_hip_pitch_link.STL; visual mesh filename=package://g1_description/meshes/right_hip_pitch_link.STL
- link right_hip_roll_link: geometry collision mesh filename=package://g1_description/meshes/right_hip_roll_link.STL; visual mesh filename=package://g1_description/meshes/right_hip_roll_link.STL
- link right_hip_yaw_link: geometry collision mesh filename=package://g1_description/meshes/right_hip_yaw_link.STL; visual mesh filename=package://g1_description/meshes/right_hip_yaw_link.STL
- link right_knee_link: geometry collision mesh filename=package://g1_description/meshes/right_knee_link.STL; visual mesh filename=package://g1_description/meshes/right_knee_link.STL
- link right_rubber_hand: geometry visual mesh filename=package://g1_description/meshes/right_rubber_hand.STL
- link right_shoulder_pitch_link: geometry collision cylinder length=0.05 radius=0.03; visual mesh filename=package://g1_description/meshes/right_shoulder_pitch_link.S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
- link right_shoulder_roll_link: geometry collision cylinder length=0.03 radius=0.03; visual mesh filename=package://g1_description/meshes/right_shoulder_roll_link.STL
- link right_shoulder_yaw_link: geometry collision mesh filename=package://g1_description/meshes/right_shoulder_yaw_link.STL; visual mesh filename=package://g1_description/meshes/right_shoulder_yaw_link.STL
- link right_wrist_pitch_link: geometry collision mesh filename=package://g1_description/meshes/right_wrist_pitch_link.STL; visual mesh filename=package://g1_description/meshes/right_wrist_pitch_link.STL
- link right_wrist_roll_link: geometry collision mesh filename=package://g1_description/meshes/right_wrist_roll_link.STL; visual mesh filename=package://g1_description/meshes/right_wrist_roll_link.STL
- link right_wrist_yaw_link: geometry collision mesh filename=package://g1_description/meshes/right_wrist_yaw_link.STL; visual mesh filename=package://g1_description/meshes/right_wrist_yaw_link.STL
- link torso_link: geometry collision mesh filename=package://g1_description/meshes/torso_link.STL; visual mesh filename=package://g1_description/meshes/torso_link.STL
- link waist_roll_link: geometry visual mesh filename=package://g1_description/meshes/waist_roll_link.STL
- link waist_support_link: geometry collision mesh filename=package://g1_description/meshes/waist_support_link.STL; visual mesh filename=package://g1_description/meshes/waist_support_link.STL
- link waist_yaw_link: geometry visual mesh filename=package://g1_description/meshes/waist_yaw_link.STL
Joints:
- removed joint d435_joint
- removed joint mid360_joint
- added joint base_joint: type fixed, parent world, child pelvis, origin xyz=0 0 0.5 rpy=0 0 0
- joint waist_yaw_joint: origin xyz=0 0 0 rpy=0 0 0 -> xyz=0 0 .01 rpy=0 0 0

File: robots/g1_description/g1_29dof_with_hand.urdf (robot description, URDF)
Before this commit: robot g1_29dof_with_hand, 53 links, 52 joints
Links:
- removed link d435_link
- removed link mid360_link
- link head_link: geometry collision mesh filename=/home/heatheramistani/Desktop/new_workspace/catkin_ws/src/u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; visual mesh filename=/home/heatheramistani/Desktop/new_workspace/catkin_ws/src/u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
- link left_ankle_pitch_link: geometry collision mesh filename=/home/heatheramistani/Desktop/new_workspace/catkin_ws/src/u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; visual mesh filename=/home/heatheramistani/Desktop/new_workspace/catkin_ws/src/u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
- link left_ankle_roll_link: geometry collision sphere radius=0.005; collision sphere radius=0.005
- link left_elbow_link: geometry collision mesh filename=/home/heatheramistani/Desktop/new_workspace/catkin_ws/src/u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; visual mesh filename=/home/heatheramistani/Desktop/new_workspace/catkin_ws/src/u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
- link left_hand_index_0_link: mass 0.05885070 -> 0.05619628; geometry collision mesh filename=/home/heatheramistani/Desktop/new_workspace/catkin_ws/src/u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; visual mesh filename=/home/heatheramistani/Desktop/new_workspace/catkin_ws/src/u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
- link left_hand_index_1_link: mass 0.02030626 -> 0.02487314; geometry collision mesh filename=/home/heatheramistani/Desktop/new_workspace/catkin_ws/src/u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; visual mesh filename=/home/heatheramistani/Desktop/new_workspace/catkin_ws/src/u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
- link left_hand_middle_0_link: mass 0.05885070 -> 0.05619628; geometry collision mesh filename=/home/heatheramistani/Desktop/new_workspace/catkin_ws/src/u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; visual mesh filename=/home/heatheramistani/Desktop/new_workspace/catkin_ws/src/u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
- link left_hand_middle_1_link: mass 0.02030626 -> 0.02487314; geometry collision mesh filename=/home/heatheramistani/Desktop/new_workspace/catkin_ws/src/u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; visual mesh filename=/home/heatheramistani/Desktop/new_workspace/catkin_ws/src/u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
- link left_hand_palm_link: geometry collision mesh filename=/home/heatheramistani/Desktop/new_workspace/catkin_ws/src/u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; visual mesh filename=/home/heatheramistani/Desktop/new_workspace/catkin_ws/src/u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
- link left_hand_thumb_0_link: mass 0.08623657 -> 0.08033018; geometry collision mesh filename=/home/heatheramistani/Desktop/new_workspace/catkin_ws/src/u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; visual mesh filename=/home/heatheramistani/Desktop/new_workspace/catkin_ws/src/u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
- link left_hand_thumb_1_link: mass 0.05885070 -> 0.05619628; geometry collision box size=0.02 0.03 0.02; visual mesh filename=/home/heatheramistani/Desktop/new_workspace/catkin_ws/src/u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
- link left_hand_thumb_2_link: mass 0.02030626 -> 0.02487314; geometry collision mesh filename=/home/heatheramistani/Desktop/new_workspace/catkin_ws/src/u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; visual mesh filename=/home/heatheramistani/Desktop/new_workspace/catkin_ws/src/u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
- link left_hip_pitch_link: geometry collision mesh filename=/home/heatheramistani/Desktop/new_workspace/catkin_ws/src/u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; visual mesh filename=/home/heatheramistani/Desktop/new_workspace/catkin_ws/src/u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
- link left_hip_roll_link: geometry collision mesh filename=/home/heatheramistani/Desktop/new_workspace/catkin_ws/src/u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; visual mesh filename=/home/heatheramistani/Desktop/new_workspace/catkin_ws/src/u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
- link left_hip_yaw_link: geometry collision mesh filename=/home/heatheramistani/Desktop/new_workspace/catkin_ws/src/u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; visual mesh filename=/home/heatheramistani/Desktop/new_workspace/catkin_ws/src/u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
- link left_knee_link: geometry collision mesh filename=/home/heatheramistani/Desktop/new_workspace/catkin_ws/src/u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; visual mesh filename=/home/heatheramistani/Desktop/new_workspace/catkin_ws/src/u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
- link left_shoulder_pitch_link: geometry collision cylinder length=0.05 radius=0.03; visual mesh filename=/home/heatheramistani/Desktop/new_workspace/catkin_ws/src/u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
- link left_shoulder_roll_link: geometry collision cylinder length=0.03 radius=0.03; visual mesh filename=/home/heatheramistani/Desktop/new_workspace/catkin_ws/src/u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
- link left_shoulder_yaw_link: geometry collision mesh filename=/home/heatheramistani/Desktop/new_workspace/catkin_ws/src/u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; visual mesh filename=/home/heatheramistani/Desktop/new_workspace/catkin_ws/src/u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
- link left_wrist_pitch_link: geometry collision mesh filename=/home/heatheramistani/Desktop/new_workspace/catkin_ws/src/u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; visual mesh filename=/home/heatheramistani/Desktop/new_workspace/catkin_ws/src/u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
- link left_wrist_roll_link: geometry collision mesh filename=/home/heatheramistani/Desktop/new_workspace/catkin_ws/src/u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; visual mesh filename=/home/heatheramistani/Desktop/new_workspace/catkin_ws/src/u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
- link left_wrist_yaw_link: geometry collision mesh filename=/home/heatheramistani/Desktop/new_workspace/catkin_ws/src/u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; visual mesh filename=/home/heatheramistani/Desktop/new_workspace/catkin_ws/src/u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
- link logo_link: geometry collision mesh filename=/home/heatheramistani/Desktop/new_workspace/catkin_ws/src/u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; visual mesh filename=/home/heatheramistani/Desktop/new_workspace/catkin_ws/src/u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
- link pelvis: geometry visual mesh filename=/home/heatheramistani/Desktop/new_workspace/catkin_ws/src/u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
- link pelvis_contour_link: geometry collision mesh filename=/home/heatheramistani/Desktop/new_workspace/catkin_ws/src/u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; visual mesh filename=/home/heatheramistani/Desktop/new_workspace/catkin_ws/src/u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
- link right_ankle_pitch_link: geometry collision mesh filename=/home/heatheramistani/Desktop/new_workspace/catkin_ws/src/u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; visual mesh filename=/home/heatheramistani/Desktop/new_workspace/catkin_ws/src/u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
- link right_ankle_roll_link: geometry collision sphere radius=0.005; collision sphere radius=0.005
- link right_elbow_link: geometry collision mesh filename=/home/heatheramistani/Desktop/new_workspace/catkin_ws/src/u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; visual mesh filename=/home/heatheramistani/Desktop/new_workspace/catkin_ws/src/u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
- link right_hand_index_0_link: mass 0.05885070 -> 0.05619628; geometry collision mesh filename=/home/heatheramistani/Desktop/new_workspace/catkin_ws/src/u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; visual mesh filename=/home/heatheramistani/Desktop/new_workspace/catkin_ws/src/u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
- link right_hand_index_1_link: mass 0.02030626 -> 0.02487314; geometry collision mesh filename=/home/heatheramistani/Desktop/new_workspace/catkin_ws/src/u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; visual mesh filename=/home/heatheramistani/Desktop/new_workspace/catkin_ws/src/u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
- link right_hand_middle_0_link: mass 0.05885070 -> 0.05619628; geometry collision mesh filename=/home/heatheramistani/Desktop/new_workspace/catkin_ws/src/u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; visual mesh filename=/home/heatheramistani/Desktop/new_workspace/catkin_ws/src/u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
- link right_hand_middle_1_link: mass 0.02030626 -> 0.02487314; geometry collision mesh filename=/home/heatheramistani/Desktop/new_workspace/catkin_ws/src/u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; visual mesh filename=/home/heatheramistani/Desktop/new_workspace/catkin_ws/src/u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
- link right_hand_palm_link: geometry collision mesh filename=/home/heatheramistani/Desktop/new_workspace/catkin_ws/src/u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; visual mesh filename=/home/heatheramistani/Desktop/new_workspace/catkin_ws/src/u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
- link right_hand_thumb_0_link: mass 0.08623657 -> 0.08033018; geometry collision mesh filename=/home/heatheramistani/Desktop/new_workspace/catkin_ws/src/u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; visual mesh filename=/home/heatheramistani/Desktop/new_workspace/catkin_ws/src/u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
- link right_hand_thumb_1_link: mass 0.05885070 -> 0.05619628; geometry collision box size=0.02 0.03 0.02; visual mesh filename=/home/heatheramistani/Desktop/new_workspace/catkin_ws/src/u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
- link right_hand_thumb_2_link: mass 0.02030626 -> 0.02487314; geometry collision mesh filename=/home/heatheramistani/Desktop/new_workspace/catkin_ws/src/u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; visual mesh filename=/home/heatheramistani/Desktop/new_workspace/catkin_ws/src/u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
- link right_hip_pitch_link: geometry collision mesh filename=/home/heatheramistani/Desktop/new_workspace/catkin_ws/src/u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; visual mesh filename=/home/heatheramistani/Desktop/new_workspace/catkin_ws/src/u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
- link right_hip_roll_link: geometry collision mesh filename=/home/heatheramistani/Desktop/new_workspace/catkin_ws/src/u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; visual mesh filename=/home/heatheramistani/Desktop/new_workspace/catkin_ws/src/u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
- link right_hip_yaw_link: geometry collision mesh filename=/home/heatheramistani/Desktop/new_workspace/catkin_ws/src/u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; visual mesh filename=/home/heatheramistani/Desktop/new_workspace/catkin_ws/src/u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
- link right_knee_link: geometry collision mesh filename=/home/heatheramistani/Desktop/new_workspace/catkin_ws/src/u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; visual mesh filename=/home/heatheramistani/Desktop/new_workspace/catkin_ws/src/u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
- link right_shoulder_pitch_link: geometry collision cylinder length=0.05 radius=0.03; visual mesh filename=/home/heatheramistani/Desktop/new_workspace/catkin_ws/src/u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
- link right_shoulder_roll_link: geometry collision cylinder length=0.03 radius=0.03; visual mesh filename=/home/heatheramistani/Desktop/new_workspace/catkin_ws/src/u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
- link right_shoulder_yaw_link: geometry collision mesh filename=/home/heatheramistani/Desktop/new_workspace/catkin_ws/src/u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; visual mesh filename=/home/heatheramistani/Desktop/new_workspace/catkin_ws/src/u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
- link right_wrist_pitch_link: geometry collision mesh filename=/home/heatheramistani/Desktop/new_workspace/catkin_ws/src/u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; visual mesh filename=/home/heatheramistani/Desktop/new_workspace/catkin_ws/src/u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
- link right_wrist_roll_link: geometry collision mesh filename=/home/heatheramistani/Desktop/new_workspace/catkin_ws/src/u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; visual mesh filename=/home/heatheramistani/Desktop/new_workspace/catkin_ws/src/u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
- link right_wrist_yaw_link: geometry collision mesh filename=/home/heatheramistani/Desktop/new_workspace/catkin_ws/src/u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; visual mesh filename=/home/heatheramistani/Desktop/new_workspace/catkin_ws/src/u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
- link torso_link: geometry collision mesh filename=/home/heatheramistani/Desktop/new_workspace/catkin_ws/src/u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; visual mesh filename=/home/heatheramistani/Desktop/new_workspace/catkin_ws/src/u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
- link waist_roll_link: geometry visual mesh filename=/home/heatheramistani/Desktop/new_workspace/catkin_ws/src/u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
- link waist_support_link: geometry collision mesh filename=/home/heatheramistani/Desktop/new_workspace/catkin_ws/src/u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; visual mesh filename=/home/heatheramistani/Desktop/new_workspace/catkin_ws/src/u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
- link waist_yaw_link: geometry visual mesh filename=/home/heatheramistani/Desktop/new_workspace/catkin_ws/src/u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
Joints:
- removed joint d435_joint
- removed joint mid360_joint
- joint left_hand_index_0_joint: limit lower=-1.57079632 upper=0 effort=1.4 velocity=12 -> lower=-1.83259571 upper=0.19198621 effort=0.7 velocity=24; origin xyz=0.0777 0.0016 0.0285 rpy=0 0 0 -> xyz=0.1 -0.0017 0.0285 rpy=0 0 0
- joint left_hand_index_1_joint: limit lower=-1.74532925 upper=0 effort=1.4 velocity=12 -> lower=-2.09439510 upper=0 effort=0.7 velocity=24; origin xyz=0.0458 0 0 rpy=0 0 0 -> xyz=0.0528 -0.0055 0 rpy=0 0 0
- joint left_hand_middle_0_joint: limit lower=-1.57079632 upper=0 effort=1.4 velocity=12 -> lower=-1.83259571 upper=0.19198621 effort=0.7 velocity=24; origin xyz=0.0777 0.0016 -0.0285 rpy=0 0 0 -> xyz=0.1 -0.0017 -0.0285 rpy=0 0 0
- joint left_hand_middle_1_joint: limit lower=-1.74532925 upper=0 effort=1.4 velocity=12 -> lower=-2.09439510 upper=0 effort=0.7 velocity=24; origin xyz=0.0458 0 0 rpy=0 0 0 -> xyz=0.0528 -0.0055 0 rpy=0 0 0
- joint left_hand_thumb_0_joint: origin xyz=0.0255 0 0 rpy=0 0 0 -> xyz=0.028 0 0 rpy=0 0 0
- joint left_hand_thumb_1_joint: limit lower=-0.72431163 upper=1.04719755 effort=1.4 velocity=12 -> lower=-0.72431163 upper=1.04719755 effort=0.7 velocity=24; origin xyz=-0.0025 -0.0193 0 rpy=0 0 0 -> xyz=0 -0.0246 0 rpy=0 0 0
- joint left_hand_thumb_2_joint: limit lower=0 upper=1.74532925 effort=1.4 velocity=12 -> lower=0 upper=2.09439510 effort=0.7 velocity=24; origin xyz=0 -0.0458 0 rpy=0 0 0 -> xyz=0.0055 -0.0528 0 rpy=0 0 0
- joint right_hand_index_0_joint: limit lower=0 upper=1.57079632 effort=1.4 velocity=12 -> lower=-0.19198621 upper=1.83259571 effort=0.7 velocity=24; origin xyz=0.0777 -0.0016 0.0285 rpy=0 0 0 -> xyz=0.1 0.0017 0.0285 rpy=0 0 0
- joint right_hand_index_1_joint: limit lower=0 upper=1.74532925 effort=1.4 velocity=12 -> lower=0 upper=2.09439510 effort=0.7 velocity=24; origin xyz=0.0458 0 0 rpy=0 0 0 -> xyz=0.0528 0.0055 0 rpy=0 0 0
- joint right_hand_middle_0_joint: limit lower=0 upper=1.57079632 effort=1.4 velocity=12 -> lower=-0.19198621 upper=1.83259571 effort=0.7 velocity=24; origin xyz=0.0777 -0.0016 -0.0285 rpy=0 0 0 -> xyz=0.1 0.0017 -0.0285 rpy=0 0 0
- joint right_hand_middle_1_joint: limit lower=0 upper=1.74532925 effort=1.4 velocity=12 -> lower=0 upper=2.09439510 effort=0.7 velocity=24; origin xyz=0.0458 0 0 rpy=0 0 0 -> xyz=0.0528 0.0055 0 rpy=0 0 0
- joint right_hand_thumb_0_joint: origin xyz=0.0255 0 0 rpy=0 0 0 -> xyz=0.028 0 0 rpy=0 0 0
- joint right_hand_thumb_1_joint: limit lower=-1.04719755 upper=0.72431163 effort=1.4 velocity=12 -> lower=-1.04719755 upper=0.72431163 effort=0.7 velocity=24; origin xyz=-0.0025 0.0193 0 rpy=0 0 0 -> xyz=0 0.0246 0 rpy=0 0 0
- joint right_hand_thumb_2_joint: limit lower=-1.74532925 upper=0 effort=1.4 velocity=12 -> lower=-2.09439510 upper=0 effort=0.7 velocity=24; origin xyz=0 0.0458 0 rpy=0 0 0 -> xyz=0.0055 0.0528 0 rpy=0 0 0

File: robots/g1_description/g1_dual_arm.urdf (robot description, URDF)
Before this commit: robot g1_dual_arm, 25 links, 24 joints
Links:
- removed link d435_link
- removed link mid360_link
Joints:
- removed joint d435_joint
- removed joint mid360_joint
