Commit message: Fixed merge

File: robots/g1_description/g1_29dof.urdf (robot description, URDF)
Before this commit: robot g1_29dof, 39 links, 38 joints
Links:
- link head_link: geometry collision mesh filename=package://meshes/head_link.STL; visual mesh filename=package://meshes/head_link.STL
- link left_ankle_pitch_link: geometry collision mesh filename=package://meshes/left_ankle_pitch_link.STL; visual mesh filename=package://meshes/left_ankle_pitch_link.STL
- link left_ankle_roll_link: geometry collision sphere radius=0.005; collision sphere radius=0.005
- link left_elbow_link: geometry collision mesh filename=package://meshes/left_elbow_link.STL; visual mesh filename=package://meshes/left_elbow_link.STL
- link left_hip_pitch_link: geometry collision mesh filename=package://meshes/left_hip_pitch_link.STL; visual mesh filename=package://meshes/left_hip_pitch_link.STL
- link left_hip_roll_link: geometry collision mesh filename=package://meshes/left_hip_roll_link.STL; visual mesh filename=package://meshes/left_hip_roll_link.STL
- link left_hip_yaw_link: geometry collision mesh filename=package://meshes/left_hip_yaw_link.STL; visual mesh filename=package://meshes/left_hip_yaw_link.STL
- link left_knee_link: geometry collision mesh filename=package://meshes/left_knee_link.STL; visual mesh filename=package://meshes/left_knee_link.STL
- link left_rubber_hand: geometry visual mesh filename=package://meshes/left_rubber_hand.STL
- link left_shoulder_pitch_link: geometry collision cylinder length=0.05 radius=0.03; visual mesh filename=package://meshes/left_shoulder_pitch_link.STL
- link left_shoulder_roll_link: geometry collision cylinder length=0.03 radius=0.03; visual mesh filename=package://meshes/left_shoulder_roll_link.STL
- link left_shoulder_yaw_link: geometry collision mesh filename=package://meshes/left_shoulder_yaw_link.STL; visual mesh filename=package://meshes/left_shoulder_yaw_link.STL
- link left_wrist_pitch_link: geometry collision mesh filename=package://meshes/left_wrist_pitch_link.STL; visual mesh filename=package://meshes/left_wrist_pitch_link.STL
- link left_wrist_roll_link: geometry collision mesh filename=package://meshes/left_wrist_roll_link.STL; visual mesh filename=package://meshes/left_wrist_roll_link.STL
- link left_wrist_yaw_link: geometry collision mesh filename=package://meshes/left_wrist_yaw_link.STL; visual mesh filename=package://meshes/left_wrist_yaw_link.STL
- link logo_link: geometry collision mesh filename=package://meshes/logo_link.STL; visual mesh filename=package://meshes/logo_link.STL
- link pelvis: geometry visual mesh filename=package://meshes/pelvis.STL
- link pelvis_contour_link: geometry collision mesh filename=package://meshes/pelvis_contour_link.STL; visual mesh filename=package://meshes/pelvis_contour_link.STL
- link right_ankle_pitch_link: geometry collision mesh filename=package://meshes/right_ankle_pitch_link.STL; visual mesh filename=package://meshes/right_ankle_pitch_link.STL
- link right_ankle_roll_link: geometry collision sphere radius=0.005; collision sphere radius=0.005
- link right_elbow_link: geometry collision mesh filename=package://meshes/right_elbow_link.STL; visual mesh filename=package://meshes/right_elbow_link.STL
- link right_hip_pitch_link: geometry collision mesh filename=package://meshes/right_hip_pitch_link.STL; visual mesh filename=package://meshes/right_hip_pitch_link.STL
- link right_hip_roll_link: geometry collision mesh filename=package://meshes/right_hip_roll_link.STL; visual mesh filename=package://meshes/right_hip_roll_link.STL
- link right_hip_yaw_link: geometry collision mesh filename=package://meshes/right_hip_yaw_link.STL; visual mesh filename=package://meshes/right_hip_yaw_link.STL
- link right_knee_link: geometry collision mesh filename=package://meshes/right_knee_link.STL; visual mesh filename=package://meshes/right_knee_link.STL
- link right_rubber_hand: geometry visual mesh filename=package://meshes/right_rubber_hand.STL
- link right_shoulder_pitch_link: geometry collision cylinder length=0.05 radius=0.03; visual mesh filename=package://meshes/right_shoulder_pitch_link.STL
- link right_shoulder_roll_link: geometry collision cylinder length=0.03 radius=0.03; visual mesh filename=package://meshes/right_shoulder_roll_link.STL
- link right_shoulder_yaw_link: geometry collision mesh filename=package://meshes/right_shoulder_yaw_link.STL; visual mesh filename=package://meshes/right_shoulder_yaw_link.STL
- link right_wrist_pitch_link: geometry collision mesh filename=package://meshes/right_wrist_pitch_link.STL; visual mesh filename=package://meshes/right_wrist_pitch_link.STL
- link right_wrist_roll_link: geometry collision mesh filename=package://meshes/right_wrist_roll_link.STL; visual mesh filename=package://meshes/right_wrist_roll_link.STL
- link right_wrist_yaw_link: geometry collision mesh filename=package://meshes/right_wrist_yaw_link.STL; visual mesh filename=package://meshes/right_wrist_yaw_link.STL
- link torso_link: geometry collision mesh filename=package://meshes/torso_link.STL; visual mesh filename=package://meshes/torso_link.STL
- link waist_roll_link: geometry visual mesh filename=package://meshes/waist_roll_link.STL
- link waist_support_link: geometry collision mesh filename=package://meshes/waist_support_link.STL; visual mesh filename=package://meshes/waist_support_link.STL
- link waist_yaw_link: geometry visual mesh filename=package://meshes/waist_yaw_link.STL

Commit message: G1 with hands and working and torso moves!

File: robots/g1_description/g1_29dof.urdf (robot description, URDF)
Before this commit: robot g1_29dof, 40 links, 39 joints
Links:
- link head_link: geometry collision mesh filename=package://g1_description/meshes/head_link.STL; visual mesh filename=package://g1_description/meshes/head_link.STL
- link left_ankle_pitch_link: geometry collision mesh filename=package://g1_description/meshes/left_ankle_pitch_link.STL; visual mesh filename=package://g1_description/meshes/left_ankle_pitch_link.STL
- link left_ankle_roll_link: geometry collision sphere radius=0.005; collision sphere radius=0.005
- link left_elbow_link: geometry collision mesh filename=package://g1_description/meshes/left_elbow_link.STL; visual mesh filename=package://g1_description/meshes/left_elbow_link.STL
- link left_hip_pitch_link: geometry collision mesh filename=package://g1_description/meshes/left_hip_pitch_link.STL; visual mesh filename=package://g1_description/meshes/left_hip_pitch_link.STL
- link left_hip_roll_link: geometry collision mesh filename=package://g1_description/meshes/left_hip_roll_link.STL; visual mesh filename=package://g1_description/meshes/left_hip_roll_link.STL
- link left_hip_yaw_link: geometry collision mesh filename=package://g1_description/meshes/left_hip_yaw_link.STL; visual mesh filename=package://g1_description/meshes/left_hip_yaw_link.STL
- link left_knee_link: geometry collision mesh filename=package://g1_description/meshes/left_knee_link.STL; visual mesh filename=package://g1_description/meshes/left_knee_link.STL
- link left_rubber_hand: geometry visual mesh filename=package://g1_description/meshes/left_hand_palm_joint.STL
- link left_shoulder_pitch_link: geometry collision cylinder length=0.05 radius=0.03; visual mesh filename=package://g1_description/meshes/left_shoulder_pitch_link.STL
- link left_shoulder_roll_link: geometry collision cylinder length=0.03 radius=0.03; visual mesh filename=package://g1_description/meshes/left_shoulder_roll_link.STL
- link left_shoulder_yaw_link: geometry collision mesh filename=package://g1_description/meshes/left_shoulder_yaw_link.STL; visual mesh filename=package://g1_description/meshes/left_shoulder_yaw_link.STL
- link left_wrist_pitch_link: geometry collision mesh filename=package://g1_description/meshes/left_wrist_pitch_link.STL; visual mesh filename=package://g1_description/meshes/left_wrist_pitch_link.STL
- link left_wrist_roll_link: geometry collision mesh filename=package://g1_description/meshes/left_wrist_roll_link.STL; visual mesh filename=package://g1_description/meshes/left_wrist_roll_link.STL
- link left_wrist_yaw_link: geometry collision mesh filename=package://g1_description/meshes/left_wrist_yaw_link.STL; visual mesh filename=package://g1_description/meshes/left_wrist_yaw_link.STL
- link logo_link: geometry collision mesh filename=package://g1_description/meshes/.STL; visual mesh filename=package://g1_description/meshes/logo_link.STL
- link pelvis: geometry visual mesh filename=package://g1_description/meshes/pelvis.STL
- link pelvis_contour_link: geometry collision mesh filename=package://g1_description/meshes/pelvis_contour_link.STL; visual mesh filename=package://g1_description/meshes/pelvis_contour_link.STL
- link right_ankle_pitch_link: geometry collision mesh filename=package://g1_description/meshes/right_ankle_pitch_link.STL; visual mesh filename=package://g1_description/meshes/right_ankle_pitch_link.STL
- link right_ankle_roll_link: geometry collision sphere radius=0.005; collision sphere radius=0.005
- link right_elbow_link: geometry collision mesh filename=package://g1_description/meshes/right_elbow_link.STL; visual mesh filename=package://g1_description/meshes/right_elbow_link.STL
- link right_hip_pitch_link: geometry collision mesh filename=package://g1_description/meshes/right_hip_pitch_link.STL; visual mesh filename=package://g1_description/meshes/right_hip_pitch_link.STL
- link right_hip_roll_link: geometry collision mesh filename=package://g1_description/meshes/right_hip_roll_link.STL; visual mesh filename=package://g1_description/meshes/right_hip_roll_link.STL
- link right_hip_yaw_link: geometry collision mesh filename=package://g1_description/meshes/right_hip_yaw_link.STL; visual mesh filename=package://g1_description/meshes/right_hip_yaw_link.STL
- link right_knee_link: geometry collision mesh filename=package://g1_description/meshes/right_knee_link.STL; visual mesh filename=package://g1_description/meshes/right_knee_link.STL
- link right_rubber_hand: geometry visual mesh filename=package://g1_description/meshes/right_rubber_hand.STL
- link right_shoulder_pitch_link: geometry collision cylinder length=0.05 radius=0.03; visual mesh filename=package://g1_description/meshes/right_shoulder_pitch_link.S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
- link right_shoulder_roll_link: geometry collision cylinder length=0.03 radius=0.03; visual mesh filename=package://g1_description/meshes/right_shoulder_roll_link.STL
- link right_shoulder_yaw_link: geometry collision mesh filename=package://g1_description/meshes/right_shoulder_yaw_link.STL; visual mesh filename=package://g1_description/meshes/right_shoulder_yaw_link.STL
- link right_wrist_pitch_link: geometry collision mesh filename=package://g1_description/meshes/right_wrist_pitch_link.STL; visual mesh filename=package://g1_description/meshes/right_wrist_pitch_link.STL
- link right_wrist_roll_link: geometry collision mesh filename=package://g1_description/meshes/right_wrist_roll_link.STL; visual mesh filename=package://g1_description/meshes/right_wrist_roll_link.STL
- link right_wrist_yaw_link: geometry collision mesh filename=package://g1_description/meshes/right_wrist_yaw_link.STL; visual mesh filename=package://g1_description/meshes/right_wrist_yaw_link.STL
- link torso_link: geometry collision mesh filename=package://g1_description/meshes/torso_link.STL; visual mesh filename=package://g1_description/meshes/torso_link.STL
- link waist_roll_link: geometry visual mesh filename=package://g1_description/meshes/waist_roll_link.STL
- link waist_support_link: geometry collision mesh filename=package://g1_description/meshes/waist_support_link.STL; visual mesh filename=package://g1_description/meshes/waist_support_link.STL
- link waist_yaw_link: geometry visual mesh filename=package://g1_description/meshes/waist_yaw_link.STL

File: robots/g1_description/g1_29dof_lock_waist.urdf (robot description, URDF)
Before this commit: robot g1_29dof_lock_waist, 40 links, 39 joints
Links:
- removed link left_ankle_pitch_link
- removed link left_ankle_roll_link
- removed link left_hip_pitch_link
- removed link left_hip_roll_link
- removed link left_hip_yaw_link
- removed link left_knee_link
- removed link right_ankle_pitch_link
- removed link right_ankle_roll_link
- removed link right_hip_pitch_link
- removed link right_hip_roll_link
- removed link right_hip_yaw_link
- removed link right_knee_link
- link head_link: geometry collision mesh filename=package://g1_description/meshes/head_link.STL; visual mesh filename=package://g1_description/meshes/head_link.STL
- link left_elbow_link: geometry collision mesh filename=package://g1_description/meshes/left_elbow_link.STL; visual mesh filename=package://g1_description/meshes/left_elbow_link.STL
- link left_rubber_hand: geometry visual mesh filename=package://g1_description/meshes/left_rubber_hand.STL
- link left_shoulder_pitch_link: geometry collision cylinder length=0.05 radius=0.03; visual mesh filename=package://g1_description/meshes/left_shoulder_pitch_link.STL
- link left_shoulder_roll_link: geometry collision cylinder length=0.03 radius=0.03; visual mesh filename=package://g1_description/meshes/left_shoulder_roll_link.STL
- link left_shoulder_yaw_link: geometry collision mesh filename=package://g1_description/meshes/left_shoulder_yaw_link.STL; visual mesh filename=package://g1_description/meshes/left_shoulder_yaw_link.STL
- link left_wrist_pitch_link: geometry collision mesh filename=package://g1_description/meshes/left_wrist_pitch_link.STL; visual mesh filename=package://g1_description/meshes/left_wrist_pitch_link.STL
- link left_wrist_roll_link: geometry collision mesh filename=package://g1_description/meshes/left_wrist_roll_link.STL; visual mesh filename=package://g1_description/meshes/left_wrist_roll_link.STL
- link left_wrist_yaw_link: geometry collision mesh filename=package://g1_description/meshes/left_wrist_yaw_link.STL; visual mesh filename=package://g1_description/meshes/left_wrist_yaw_link.STL
- link logo_link: geometry collision mesh filename=package://g1_description/meshes/logo_link.STL; visual mesh filename=package://g1_description/meshes/logo_link.STL
- link pelvis: geometry visual mesh filename=package://g1_description/meshes/pelvis.STL
- link pelvis_contour_link: geometry collision mesh filename=package://g1_description/meshes/pelvis_contour_link.STL; visual mesh filename=package://g1_description/meshes/pelvis_contour_link.STL
- link right_elbow_link: geometry collision mesh filename=package://g1_description/meshes/right_elbow_link.STL; visual mesh filename=package://g1_description/meshes/right_elbow_link.STL
- link right_rubber_hand: geometry visual mesh filename=package://g1_description/meshes/right_rubber_hand.STL
- link right_shoulder_pitch_link: geometry collision cylinder length=0.05 radius=0.03; visual mesh filename=package://g1_description/meshes/right_shoulder_pitch_link.S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
- link right_shoulder_roll_link: geometry collision cylinder length=0.03 radius=0.03; visual mesh filename=package://g1_description/meshes/right_shoulder_roll_link.STL
- link right_shoulder_yaw_link: geometry collision mesh filename=package://g1_description/meshes/right_shoulder_yaw_link.STL; visual mesh filename=package://g1_description/meshes/right_shoulder_yaw_link.STL
- link right_wrist_pitch_link: geometry collision mesh filename=package://g1_description/meshes/right_wrist_pitch_link.STL; visual mesh filename=package://g1_description/meshes/right_wrist_pitch_link.STL
- link right_wrist_roll_link: geometry collision mesh filename=package://g1_description/meshes/right_wrist_roll_link.STL; visual mesh filename=package://g1_description/meshes/right_wrist_roll_link.STL
- link right_wrist_yaw_link: geometry collision mesh filename=package://g1_description/meshes/right_wrist_yaw_link.STL; visual mesh filename=package://g1_description/meshes/right_wrist_yaw_link.STL
- link torso_link: geometry collision mesh filename=package://g1_description/meshes/torso_link.STL; visual mesh filename=package://g1_description/meshes/torso_link.STL
- link waist_roll_link: geometry visual mesh filename=package://g1_description/meshes/waist_roll_link.STL
- link waist_support_link: geometry collision mesh filename=package://g1_description/meshes/waist_support_link.STL; visual mesh filename=package://g1_description/meshes/waist_support_link.STL
- link waist_yaw_link: geometry visual mesh filename=package://g1_description/meshes/waist_yaw_link.STL
Joints:
- removed joint left_ankle_pitch_joint
- removed joint left_ankle_roll_joint
- removed joint left_hip_pitch_joint
- removed joint left_hip_roll_joint
- removed joint left_hip_yaw_joint
- removed joint left_knee_joint
- removed joint right_ankle_pitch_joint
- removed joint right_ankle_roll_joint
- removed joint right_hip_pitch_joint
- removed joint right_hip_roll_joint
- removed joint right_hip_yaw_joint
- removed joint right_knee_joint
